File: AudioAmplifier-1.kicad_pcb (KiCad board)
At the start: 2 copper layers, 64.8 x 41.3 mm, 25 parts, among them J1 Conn_01x03, J2 Conn_01x03, J3 Conn_01x02, J4 Conn_01x04, Q1 Q_NPN_EBC, U1 LM386, U2 MCP41010

Commit message: Improved layout
Parts:
- removed the REF** at (165.7, 111.1)
- added C9: 0.1u, kc1fsz-footprint-library:C_Disc_D4.7mm_W2.5mm_P5.00mm, F.Cu at (137.2, 113.0)
- added J5: Conn_01x01, Connectors:1pin, F.Cu at (165.7, 111.1)
- C1, C4: value C -> 1u; footprint Capacitors_THT:C_Disc_D10.5mm_W5.0mm_P7.50mm -> Capacitors_THT:CP_Radial_D5.0mm_P2.50mm
- C3: footprint Capacitors_THT:C_Disc_D10.5mm_W5.0mm_P7.50mm -> kc1fsz-footprint-library:C_Disc_D4.7mm_W2.5mm_P5.00mm
- C5: footprint Capacitors_THT:CP_Radial_D5.0mm_P2.50mm -> Capacitors_THT:CP_Radial_D10.0mm_P5.00mm
- C7: value C -> 0.1u; footprint Capacitors_THT:C_Disc_D10.5mm_W5.0mm_P7.50mm -> kc1fsz-footprint-library:C_Disc_D4.7mm_W2.5mm_P5.00mm
- C8: value CP -> 470u
- R5: value R -> 10
- U2: value MCP41010 -> MCP4131-103
- moved C6 5.46 mm to (154.9, 80.0)
- moved C5 3.70 mm to (147.3, 78.7)
- moved J3 0.63 mm to (161.3, 82.5)
Connections:
- C4 pad 1: Net-(C4-Pad1) -> Net-(C3-Pad1)
- C4 pad 2: Net-(C3-Pad1) -> Net-(C4-Pad2)
- J2 pad 1: Net-(C4-Pad1) -> Net-(C4-Pad2)
- U2 pad 5: Net-(C4-Pad1) -> Net-(C4-Pad2)
Routing:
- net Net-(C4-Pad2): track 0.00 -> 44.0 mm
- net Net-(C4-Pad1): track 32.2 -> 0.00 mm
- net Net-(C1-Pad1): track 36.7 -> 25.7 mm
- net Net-(C5-Pad1): track 24.5 -> 32.3 mm
- net Net-(C6-Pad2): track 7.91 -> 14.0 mm
- net Net-(C6-Pad1): track 11.5 -> 17.7 mm
- net Net-(C1-Pad2): track 7.26 -> 12.3 mm
- net Net-(C9-Pad1): track 23.0 -> 27.1 mm
- net Net-(C3-Pad1): track 30.7 -> 27.2 mm
- net Net-(J2-Pad2): track 22.4 -> 20.6 mm
- net Net-(J4-Pad2): track 16.7 -> 18.2 mm
- net Net-(J4-Pad1): track 23.2 -> 24.1 mm
Other:
- net class Default: clearance 0.01 -> 0.254; trace_width 0.91 -> 0.254; via_dia 0.027 -> 0.6858; via_drill 0.013 -> 0.3302
- rule trace_clearance: 0.01 -> 0.254
- rule trace_min: 0.01 -> 0.254
- rule via_min_drill: 0.013 -> 0.3302
- rule via_min_size: 0.027 -> 0.6858
- board text added: "2018-06 v2"
- board text added: "KC1FSZ"
- board text removed: "KC1FSZ v1"
